File: usb.sch (KiCad schematic (older format))
At the start: 92 parts, among them J201 USB_B, J202 CONN_ICSP, J203 CONN_MRESET, J204 CONN_LED, SW201 SW_RESET, U201 ATmega32U4-AU, U202 MAX7221, Y201 16M, Y202 16M

Commit message: Happy?
Parts:
- removed LD7:4: LED_SPC, LED_THT:LED_D3.0mm, symbol Device:LED
- added LD1B:7: LED_RSH, LED_THT:LED_D3.0mm, symbol Device:LED
- added LD7A:4: LED_SPC1, LED_THT:LED_D3.0mm, symbol Device:LED
- added LD7B:4: LED_SPC2, LED_THT:LED_D3.0mm, symbol Device:LED
- added LD7C:4: LED_SPC3, LED_THT:LED_D3.0mm, symbol Device:LED
- added Q201, Q202: MMBT3904, Package_TO_SOT_SMD:SOT-23, symbol Device:Q_NPN_BEC
- added R5, R6, R7, R8, R9: 1k, Resistor_SMD:R_0805_2012Metric_Pad1.20x1.40mm_HandSolder, symbol Device:R
- renumbered LD1:7 to LD1A:7
Connections:
- net +5V: now also Q201.3 (C), Q202.3 (C)
- net lcol4: now also R7.1, R8.1, R9.1
- net lcol7: now also R5.1, R6.1; no longer LD1A:7.1 (K)
- net lrow1: now also Q201.1 (B); no longer LD1A:7.2 (A)
- net lrow7: now also Q202.1 (B)
- new net: LD1B:7.1 (K), R6.2
- new net: LD1A:7.2 (A), LD1B:7.2 (A), Q201.2 (E)
- new net: LD1A:7.1 (K), R5.2
- new net: LD7A:4.1 (K), R7.2
- new net: LD7A:4.2 (A), LD7B:4.2 (A), LD7C:4.2 (A), Q202.2 (E)
- new net: LD7B:4.1 (K), R8.2
- new net: LD7C:4.1 (K), R9.2
Other:
- note added: "Hack to light up several leds\nat a single matrix point\nThanks @Mattman944!"
- moved on the sheet: LD0:0, LD0:1, LD0:2, LD0:3, LD0:4, LD0:5, LD0:6, LD0:7, LD1:0, LD1:1, LD1:2, LD1:3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

Commit message: IN PRODUCTION!
Parts:
- C201, C202: LCSC C1797 -> C1804
- C203: LCSC C16133 -> (none)
- D201: value 1n4148 -> 1n5819; footprint Diode_SMD:D_SOD-323_HandSoldering -> Diode_SMD:D_SMA; LCSC C2128 -> C191023
- J201: LCSC C397338 -> (none)
- LD0:0, LD0:1, LD0:2, LD0:3, LD0:4, LD0:5, LD0:6, LD0:7, LD1:0, LD1:1, LD1:2, LD1:3, LD1:4, LD1:5, LD1:6, LD1A:7, LD1B:7, LD2:0, LD2:1, LD2:2, LD2:3, LD2:4, LD2:5, LD2:6, LD2:7, LD3:0, LD3:1, LD3:2, LD3:3, LD3:4, LD3:5, LD3:6, LD3:7, LD4:0, LD4:1, LD4:2, LD4:3, LD4:4, LD4:5, LD4:6, LD4:7, LD5:0, LD5:1, LD5:2, LD5:3, LD5:4, LD5:5, LD5:6, LD5:7, LD6:0, LD6:1, LD6:2, LD6:3, LD6:4, LD6:5, LD6:6, LD6:7, LD7:0, LD7:1, LD7:2, LD7:3, LD7:5, LD7:6, LD7:7, LD7A:4, LD7B:4, LD7C:4: LCSC C2297 -> (none)
- Q201, Q202: LCSC (none) -> C20526
- R207: value 22k -> 220k; LCSC C17414 -> C17556
- SW201: LCSC C410365 -> C318884
- renumbered R7 to R208, R8 to R209, R9 to R210, R5 to R211, R6 to R212

Commit message: Make 1u caps uniform
Parts:
- removed C204: 1u, Capacitor_THT:CP_Radial_D5.0mm_P2.00mm, symbol Device:C
- added C204: 1u, Capacitor_THT:CP_Radial_D5.0mm_P2.00mm, symbol Device:CP1
Connections:
- net GND: now also C204.2
- net at U201.6 (UCAP): now also C204.1
Changed lines of the file:
@@
-$EndComp
-$Comp
-L Device:C C204
-U 1 1 5E637503
-P 1785 3770
-F 0 "C204" H 1900 3816 50  0000 L CNN
-F 1 "1u" H 1900 3725 50  0000 L CNN
-F 2 "Capacitor_THT:CP_Radial_D5.0mm_P2.00mm" H 1823 3620 50  0001 C CNN
-F 3 "~" H 1785 3770 50  0001 C CNN
-F 4 "C1848" H 1785 3770 50  0001 C CNN "LCSC"
-	1    1785 3770
-	1    0    0    -1
 $EndComp
 $Comp
@@
 Text Notes 14195 2935 0    50   ~ 0
 Hack to light up several leds\nat a single matrix point\nThanks @Mattman944!
+$Comp
+L Device:CP1 C204
+U 1 1 66DA4E1C
+P 1785 3770
+F 0 "C204" H 1900 3816 50  0000 L CNN
+F 1 "1u" H 1900 3725 50  0000 L CNN
+F 2 "Capacitor_THT:CP_Radial_D5.0mm_P2.00mm" H 1785 3770 50  0001 C CNN
+F 3 "~" H 1785 3770 50  0001 C CNN
+	1    1785 3770
+	1    0    0    -1
+$EndComp
 Wire Bus Line
 	3930 2075 3930 2775
